Commit message: moveit config ready

File: mit_robot_description/urdf/mit_robot.urdf.xacro (robot description, xacro)
@@ -7,4 +7,5 @@
 	 <xacro:arg name="name" default="ur"/>
    <xacro:arg name="ur_type" default="ur5e"/>
+	 <xacro:arg name="prefix" default=""/>
 	 <xacro:arg name="sim_gazebo" default="true" />
 	 <xacro:arg name="simulation_controllers" default="$(find mit_robot_control)/config/ur_controllers.yaml" />

File: mit_robot_moveit_config/config/ur.ros2_control.xacro (robot description, xacro)
@@ -1,6 +1,6 @@
 <?xml version="1.0"?>
 <robot xmlns:xacro="http://www.ros.org/wiki/xacro">
-    <xacro:macro name="mit_robot_ros2_control" params="name">
-        <!-- <xacro:property name="initial_positions" value="${load_yaml(initial_positions_file)['initial_positions']}"/> -->
+    <xacro:macro name="ur_ros2_control" params="name initial_positions_file">
+        <xacro:property name="initial_positions" value="${load_yaml(initial_positions_file)['initial_positions']}"/>
         <ros2_control name="${name}" type="system">
             <hardware>
@@ -11,5 +11,5 @@
                 <command_interface name="position"/>
                 <state_interface name="position">
-                  <param name="initial_value">0</param>
+                  <param name="initial_value">${initial_positions['shoulder_pan_joint']}</param>
                 </state_interface>
                 <state_interface name="velocity"/>
@@ -18,5 +18,5 @@
                 <command_interface name="position"/>
                 <state_interface name="position">
-                  <param name="initial_value">-1.5707</param>
+                  <param name="initial_value">${initial_positions['shoulder_lift_joint']}</param>
                 </state_interface>
                 <state_interface name="velocity"/>
@@ -25,5 +25,5 @@
                 <command_interface name="position"/>
                 <state_interface name="position">
-                  <param name="initial_value">0</param>
+                  <param name="initial_value">${initial_positions['elbow_joint']}</param>
                 </state_interface>
                 <state_interface name="velocity"/>
@@ -32,5 +32,5 @@
                 <command_interface name="position"/>
                 <state_interface name="position">
-                  <param name="initial_value">0</param>
+                  <param name="initial_value">${initial_positions['wrist_1_joint']}</param>
                 </state_interface>
                 <state_interface name="velocity"/>
@@ -39,5 +39,5 @@
                 <command_interface name="position"/>
                 <state_interface name="position">
-                  <param name="initial_value">0</param>
+                  <param name="initial_value">${initial_positions['wrist_2_joint']}</param>
                 </state_interface>
                 <state_interface name="velocity"/>
@@ -46,5 +46,5 @@
                 <command_interface name="position"/>
                 <state_interface name="position">
-                  <param name="initial_value">0</param>
+                  <param name="initial_value">${initial_positions['wrist_3_joint']}</param>
                 </state_interface>
                 <state_interface name="velocity"/>

Commit message: Added gripper

File: mit_robot_description/urdf/mit_robot.urdf.xacro (robot description, xacro)
@@ -1,14 +1,18 @@
 <?xml version="1.0"?>
 <robot xmlns:xacro="http://wiki.ros.org/xacro" name="ur">
-	 <!-- xacro arguments -->
-   <xacro:arg name="safety_limits" default="true"/>
-   <xacro:arg name="safety_pos_margin" default="0.15"/>
-   <xacro:arg name="safety_k_position" default="20"/>
-	 <xacro:arg name="name" default="ur"/>
-   <xacro:arg name="ur_type" default="ur5e"/>
-	 <xacro:arg name="prefix" default=""/>
-	 <xacro:arg name="sim_gazebo" default="true" />
-	 <xacro:arg name="simulation_controllers" default="$(find mit_robot_control)/config/ur_controllers.yaml" />
-   <!-- import main macro -->
-   <xacro:include filename="$(find ur_description)/urdf/ur.urdf.xacro"/>
+	<!-- xacro arguments -->
+	<xacro:arg name="safety_limits" default="true"/>
+	<xacro:arg name="safety_pos_margin" default="0.15"/>
+	<xacro:arg name="safety_k_position" default="20"/>
+	<xacro:arg name="name" default="ur"/>
+	<xacro:arg name="ur_type" default="ur5e"/>
+	<xacro:arg name="prefix" default=""/>
+	<xacro:arg name="sim_gazebo" default="true" />
+	<xacro:arg name="simulation_controllers" default="$(find mit_robot_control)/config/ur_controllers.yaml" />
+	<!-- import main macro -->
+	<xacro:include filename="$(find ur_description)/urdf/ur.urdf.xacro"/>
+	<!-- add materials -->
+	<xacro:include filename="$(find mit_robot_description)/urdf/materials.urdf.xacro"/>
+	 <!-- add gripper -->
+	<xacro:include filename="$(find mit_robot_description)/urdf/gripper.urdf.xacro"/>
 </robot>

File: mit_robot_moveit_config/config/ur.ros2_control.xacro (robot description, xacro)
@@ -1,6 +1,5 @@
 <?xml version="1.0"?>
 <robot xmlns:xacro="http://www.ros.org/wiki/xacro">
-    <xacro:macro name="ur_ros2_control" params="name initial_positions_file">
-        <xacro:property name="initial_positions" value="${load_yaml(initial_positions_file)['initial_positions']}"/>
+    <xacro:macro name="ur_ros2_control" params="name">
         <ros2_control name="${name}" type="system">
             <hardware>
@@ -11,5 +10,5 @@
                 <command_interface name="position"/>
                 <state_interface name="position">
-                  <param name="initial_value">${initial_positions['shoulder_pan_joint']}</param>
+                  <param name="initial_value">0</param>
                 </state_interface>
                 <state_interface name="velocity"/>
@@ -18,5 +17,5 @@
                 <command_interface name="position"/>
                 <state_interface name="position">
-                  <param name="initial_value">${initial_positions['shoulder_lift_joint']}</param>
+                  <param name="initial_value">0</param>
                 </state_interface>
                 <state_interface name="velocity"/>
@@ -25,5 +24,5 @@
                 <command_interface name="position"/>
                 <state_interface name="position">
-                  <param name="initial_value">${initial_positions['elbow_joint']}</param>
+                  <param name="initial_value">0</param>
                 </state_interface>
                 <state_interface name="velocity"/>
@@ -32,5 +31,5 @@
                 <command_interface name="position"/>
                 <state_interface name="position">
-                  <param name="initial_value">${initial_positions['wrist_1_joint']}</param>
+                  <param name="initial_value">0</param>
                 </state_interface>
                 <state_interface name="velocity"/>
@@ -39,5 +38,5 @@
                 <command_interface name="position"/>
                 <state_interface name="position">
-                  <param name="initial_value">${initial_positions['wrist_2_joint']}</param>
+                  <param name="initial_value">0</param>
                 </state_interface>
                 <state_interface name="velocity"/>
@@ -46,5 +45,5 @@
                 <command_interface name="position"/>
                 <state_interface name="position">
-                  <param name="initial_value">${initial_positions['wrist_3_joint']}</param>
+                  <param name="initial_value">0</param>
                 </state_interface>
                 <state_interface name="velocity"/>

File: mit_robot_moveit_config/config/ur.urdf.xacro (robot description, xacro)
@@ -1,9 +1,8 @@
 <?xml version="1.0"?>
 <robot xmlns:xacro="http://www.ros.org/wiki/xacro" name="ur">
-    <xacro:arg name="initial_positions_file" default="initial_positions.yaml" />
     <!-- Import ur urdf file -->
     <xacro:include filename="$(find mit_robot_description)/urdf/mit_robot.urdf.xacro" />
     <!-- Import control_xacro -->
     <xacro:include filename="ur.ros2_control.xacro" />
-    <xacro:ur_ros2_control name="FakeSystem" initial_positions_file="$(arg initial_positions_file)"/>
+    <xacro:ur_ros2_control name="FakeSystem"/>
 </robot>

File: mit_robot_moveit_config/srdf/mit_robot_macro.srdf.xacro (robot description, xacro)
@@ -53,4 +53,5 @@
     <disable_collisions link1="${prefix}wrist_1_link" link2="${prefix}wrist_3_link" reason="Never" />
     <disable_collisions link1="${prefix}wrist_2_link" link2="${prefix}wrist_3_link" reason="Adjacent" />
+    <disable_collisions link1="suction_gripper_link" link2="wrist_3_link" reason="Adjacent"/>
   </xacro:macro>
 </robot>
