Commit message: Added gripper plugin

File: mit_robot_description/urdf/gripper.urdf.xacro (robot description, xacro)
@@ -1,5 +1,5 @@
 <?xml version="1.0"?>
 <robot xmlns:xacro="http://wiki.ros.org/xacro" name="ur">
-	<link name="suction_gripper_link">
+	<link name="suction_base_link">
 		<inertial>
 			<origin xyz="0 0 -0.026287" rpy="0 0 0"/>
@@ -21,11 +21,21 @@
 		</visual>
 	</link>
-	<gazebo reference="suction_gripper_link">
-		<material>Gazebo/White</material>
-	</gazebo>
 	<joint name="gripper_joint" type="fixed">
 		<parent link="tool0"/>
-		<child link="suction_gripper_link"/>
+		<child link="suction_base_link"/>
 		<origin xyz="0 0 0" rpy="0 ${pi} 0"/>
 	</joint>
+	<!-- Adding link for gripping -->
+	<link name="suction_gripper_link">
+		<inertial>
+			<mass value="0.001"/>
+			<inertia ixx="1e-6" ixy="0.0" ixz="0.0" iyy="1e-6" iyz="0.0" izz="1e-6"/>
+		</inertial>
+	</link>
+	<joint name="suction_gripper_joint" type="continuous">
+		<parent link="wrist_3_link"/>
+		<child link="suction_gripper_link"/>
+		<origin xyz="0 0 0.1" rpy="0 ${-pi/2} ${pi}"/>
+		<axis xyz="0 0 1" rpy="0 0 0" />
+	</joint>
 </robot>

File: mit_robot_description/urdf/mit_robot.urdf.xacro (robot description, xacro)
@@ -16,3 +16,5 @@
 	 <!-- add gripper -->
 	<xacro:include filename="$(find mit_robot_description)/urdf/gripper.urdf.xacro"/>
+	<!-- add gazebo related -->
+	<xacro:include filename="$(find mit_robot_description)/urdf/mit_robot.gazebo.urdf.xacro"/>
 </robot>

File: mit_robot_moveit_config/srdf/mit_robot_macro.srdf.xacro (robot description, xacro)
@@ -53,5 +53,5 @@
     <disable_collisions link1="${prefix}wrist_1_link" link2="${prefix}wrist_3_link" reason="Never" />
     <disable_collisions link1="${prefix}wrist_2_link" link2="${prefix}wrist_3_link" reason="Adjacent" />
-    <disable_collisions link1="suction_gripper_link" link2="wrist_3_link" reason="Adjacent"/>
+    <disable_collisions link1="suction_base_link" link2="wrist_3_link" reason="Adjacent"/>
   </xacro:macro>
 </robot>

Commit message: Added models and configured worlds

File: mit_robot_description/urdf/gripper.urdf.xacro (robot description, xacro)
@@ -27,15 +27,9 @@
 	</joint>
 	<!-- Adding link for gripping -->
-	<link name="suction_gripper_link">
-		<inertial>
-			<mass value="0.001"/>
-			<inertia ixx="1e-6" ixy="0.0" ixz="0.0" iyy="1e-6" iyz="0.0" izz="1e-6"/>
-		</inertial>
-	</link>
-	<joint name="suction_gripper_joint" type="continuous">
-		<parent link="wrist_3_link"/>
+	<link name="suction_gripper_link"/>
+	<joint name="suction_gripper_joint" type="fixed">
+		<parent link="suction_base_link"/>
 		<child link="suction_gripper_link"/>
-		<origin xyz="0 0 0.1" rpy="0 ${-pi/2} ${pi}"/>
-		<axis xyz="0 0 1" rpy="0 0 0" />
+		<origin xyz="0 0 -0.1" rpy="0 0 0"/>
 	</joint>
 </robot>

File: mit_robot_description/urdf/mit_robot.gazebo.urdf.xacro (robot description, xacro)
@@ -11,5 +11,5 @@
 				<remapping>grasping:=grasping_test</remapping>
 			</ros>
-			<link_name>suction_gripper_link</link_name>
+			<link_name>wrist_3_link</link_name>
 			<max_distance>10.0</max_distance>
 			<fixed>ground_plane</fixed>

Commit message: Added planning group

File: mit_robot_description/urdf/gripper.urdf.xacro (robot description, xacro)
@@ -21,15 +21,31 @@
 		</visual>
 	</link>
-	<joint name="gripper_joint" type="fixed">
-		<parent link="tool0"/>
-		<child link="suction_base_link"/>
-		<origin xyz="0 0 0" rpy="0 ${pi} 0"/>
+	<joint name="suction_base_joint" type="revolute">
+		<axis xyz="1 0 0" />
+		<parent link="wrist_3_link" />
+		<child link="suction_base_link" />
+		<origin rpy="0 ${pi} 0" xyz="0 0 0" />
+		<limit effort="50" velocity="50" lower="-${pi}" upper="${pi}" />
+		<dynamics damping="0.0" friction="10"/>
 	</joint>
-	<!-- Adding link for gripping -->
-	<link name="suction_gripper_link"/>
-	<joint name="suction_gripper_joint" type="fixed">
-		<parent link="suction_base_link"/>
-		<child link="suction_gripper_link"/>
-		<origin xyz="0 0 -0.1" rpy="0 0 0"/>
-	</joint>
+	<ros2_control name="GazeboSystem" type="system">
+    <hardware>
+      <plugin>gazebo_ros2_control/GazeboSystem</plugin>
+    </hardware>
+		<joint name="suction_base_joint">
+      <command_interface name="position"/>
+      <state_interface name="position"/>
+      <state_interface name="velocity"/>
+      <state_interface name="effort"/>
+    </joint>
+	</ros2_control>
+	<transmission name="suction_base_trans">
+		<type>transmission_interface/SimpleTransmission</type>
+		<joint name="suction_base_joint">
+			<hardwareInterface>hardware_interface/PositionJointInterface</hardwareInterface>
+		</joint>
+		<actuator name="suction_base_motor">
+			<mechanicalReduction>1</mechanicalReduction>
+		</actuator>
+	</transmission>
 </robot>

File: mit_robot_moveit_config/srdf/mit_robot_macro.srdf.xacro (robot description, xacro)
@@ -13,4 +13,7 @@
     <group name="${prefix}${name}_manipulator">
       <chain base_link="${prefix}base_link" tip_link="${prefix}tool0" />
+    </group>
+    <group name="gripper">
+        <joint name="suction_base_joint"/>
     </group>
     <!--GROUP STATES - Purpose - Define a named state for a particular group, in terms of joint values. This is useful to define states like 'folded arms'-->
@@ -39,5 +42,11 @@
       <joint name="${prefix}wrist_3_joint" value="-0.11" />
     </group_state>
-    <!--END EFFECTOR - Purpose - Represent information about an end effector.-->
+    <group_state name="open" group="gripper">
+        <joint name="suction_base_joint" value="0"/>
+    </group_state>
+    <group_state name="close" group="gripper">
+        <joint name="suction_base_joint" value="0"/>
+    </group_state>
+    <end_effector name="gripper" parent_link="wrist_3_link" group="gripper" parent_group="ur_manipulator"/>
     <!--VIRTUAL JOINT - Purpose - this element defines a virtual joint between a robot link and an external frame of reference (considered fixed with respect to the robot)-->
     <!--DISABLE COLLISIONS - By default it is assumed that any link of the robot could potentially come into collision with any other link in the robot. This tag disables collision checking between a specified pair of links. -->

Commit message: almost fixed mtc

File: mit_robot_description/urdf/gripper.urdf.xacro (robot description, xacro)
@@ -26,6 +26,6 @@
 		<child link="suction_base_link" />
 		<origin rpy="0 ${pi} 0" xyz="0 0 0" />
-		<limit effort="50" velocity="50" lower="-${pi}" upper="${pi}" />
-		<dynamics damping="0.0" friction="10"/>
+		<limit effort="50" velocity="50" lower="-${0.001}" upper="${0}" />
+		<dynamics damping="1000.0" friction="1000"/>
 	</joint>
 	<ros2_control name="GazeboSystem" type="system">

File: mit_robot_description/urdf/mit_robot.gazebo.urdf.xacro (robot description, xacro)
@@ -11,6 +11,6 @@
 				<remapping>grasping:=grasping_test</remapping>
 			</ros>
-			<link_name>wrist_3_link</link_name>
-			<max_distance>10.0</max_distance>
+			<link_name>suction_base_link</link_name>
+			<max_distance>0.2</max_distance>
 			<fixed>ground_plane</fixed>
 		</plugin>
